File: Electrical/BridgeCircuit/BridgeCircuit.kicad_sch (KiCad schematic)
At the start: 43 parts, among them M1 Motor_DC, M2 Motor_DC, M3 Motor_Servo, M4 Motor_Servo, Q1 NPN, Q2 NPN, Q3 NPN, Q4 NPN, Q5 NPN, Q6 NPN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

Commit message: Schematic V4
Parts:
- removed D1, D4: Red, symbol Device:LED
- removed D2, D5: Yellow, symbol Device:LED
- removed D3, D6: Green, symbol Device:LED
- removed R1: 70Ω, symbol Device:R_US
- removed U3: ~, symbol Custom_KiCadLibrary:ESP-WROOM-32-Devkit
- added D13, D14: Red, symbol Device:LED
- added D15, D16: Yellow, symbol Device:LED
- added D17, D18: Green, symbol Device:LED
- added R13, R14, R15, R16, R17, R18, R19: 180Ω, symbol Device:R_US
- added U6: ~, symbol Custom_KiCadLibrary:ESP-WROOM-32-Devkit_ENGG3K
- Q1, Q2, Q3, Q4, Q5, Q6: value NPN -> BC547
- R10, R11, R12, R7, R8, R9: value R_US -> 180Ω
- R2, R3, R4, R5, R6: value 70Ω -> 180Ω
Connections:
- net D34 is gone; now on net D22: R12.1
- net D35 is gone; now on net D23: R11.1
- net D5 is gone; now on net GND: U5. (Gnd)
- net +5V: now also R10.1, R8.1, R9.1, U1. (GND), R14.1, R15.1, R16.1, R17.1, R18.1, R19.1, U6. (EN); no longer R5.1, R6.1
- net D12: now also U6. (EN)
- net D13: now also U6. (EN)
- net D14: now also R6.1, U6. (EN); no longer U1. (GND)
- net D15: now also U6. (EN)
- net D18: now also U6. (EN)
- net D19: now also U6. (EN)
- net D2: now also U6. (EN)
- net D21: now also R13.1, U6. (EN); no longer R9.1
- net D22: now also U6. (EN); no longer R8.1
- net D23: now also U6. (EN); no longer R7.1
- net D25: now also U6. (EN)
- net D26: now also U6. (EN)
- net D27: now also R7.1, U6. (EN); no longer U1. (GND)
- net D32: now also R5.1, U6. (EN); no longer R10.1
- net D33: now also U6. (EN)
- net D4: now also U6. (EN)
- net GND: now also U6. (EN)
- net at D11.1 (K): now also D12.1 (K), Q6.1 (C); no longer D12.2 (A)
- net at D11.2 (A): now also R4.2; no longer R6.2
- net at D10.1 (K), Q5.1 (C): now also D9.1 (K)
- net at Q5.2 (B): now also R6.2; no longer R11.2
- net at D7.2 (A): now also R2.2; no longer R4.2
- net at R3.2: now also D9.2 (A)
- net at Q3.1 (C): now also D17.1 (K), D18.1 (K)
- net at R9.2: now also D15.2 (A); no longer Q3.2 (B)
- net at D10.2 (A): now also R15.2; no longer D9.1 (K)
- net at D7.1 (K): now also D8.1 (K), Q4.1 (C); no longer D8.2 (A)
- net at R12.2: now also Q2.2 (B); no longer Q6.2 (B)
- net at Q1.1 (C): now also D13.1 (K), D14.1 (K)
- net at Q1.2 (B): now also R11.2; no longer R7.2
- net at Q2.1 (C): now also D15.1 (K), D16.1 (K)
- net at R10.2: now also D17.2 (A); no longer Q4.2 (B)
- net at R8.2: now also D13.2 (A); no longer Q2.2 (B)
- net at R5.2: now also Q4.2 (B); no longer D9.2 (A)
- new net: D18.2 (A), R19.2
- new net: D8.2 (A), R14.2
- new net: Q3.2 (B), R13.2
- new net: Q6.2 (B), R7.2
- new net: D12.2 (A), R16.2
- new net: D16.2 (A), R18.2
- new net: D14.2 (A), R17.2
- new net D16: U5. (Gnd), U6. (EN)
Other:
- note added: "21st Oct. 2025"
- note added: "V4"
- note removed: "24th Aug. 2025"
- note removed: "V2"
- moved on the sheet: D11, D7, D9, LS1, Q1, Q2, Q3, R2, SW1
